File: PCB/main_board/main_board_schematic/main_board_schematic.kicad_sch (KiCad schematic)
At the start: 257 parts, among them J1 Conn_01x02, J2 Conn_01x02, J3 Conn_01x02, P1 USB_C_Plug_USB2.0, SW1 SW_MEC_5G, SW10 SW_MEC_5G, SW100 SW_MEC_5G, SW101 SW_MEC_5G, SW102 SW_MEC_5G, SW103 SW_MEC_5G, SW104 SW_MEC_5G, SW105 SW_MEC_5G, SW106 SW_MEC_5G, SW107 SW_MEC_5G, SW108 SW_MEC_5G, SW11 SW_MEC_5G, SW12 SW_MEC_5G, SW13 SW_MEC_5G, SW14 SW_MEC_5G, SW15 SW_MEC_5G, SW16 SW_MEC_5G, SW17 SW_MEC_5G, SW18 SW_MEC_5G, SW19 SW_MEC_5G, SW2 SW_MEC_5G, SW20 SW_MEC_5G, SW21 SW_MEC_5G, SW22 SW_MEC_5G, SW23 SW_MEC_5G, SW24 SW_MEC_5G, SW25 SW_MEC_5G, SW26 SW_MEC_5G, SW27 SW_MEC_5G, SW28 SW_MEC_5G, SW29 SW_MEC_5G, SW3 SW_MEC_5G, SW30 SW_MEC_5G, SW31 SW_MEC_5G, SW32 SW_MEC_5G, SW33 SW_MEC_5G, SW34 SW_MEC_5G, SW35 SW_MEC_5G, SW36 SW_MEC_5G, SW37 SW_MEC_5G, SW38 SW_MEC_5G, SW39 SW_MEC_5G, SW4 SW_MEC_5G, SW40 SW_MEC_5G, SW41 SW_MEC_5G, SW42 SW_MEC_5G, SW43 SW_MEC_5G, SW44 SW_MEC_5G, SW45 SW_MEC_5G, SW46 SW_MEC_5G, SW47 SW_MEC_5G, SW48 SW_MEC_5G, SW49 SW_MEC_5G, SW5 SW_MEC_5G, SW50 SW_MEC_5G, SW51 SW_MEC_5G, SW52 SW_MEC_5G, SW53 SW_MEC_5G, SW54 SW_MEC_5G, SW55 SW_MEC_5G, SW56 SW_MEC_5G, SW57 SW_MEC_5G, SW58 SW_MEC_5G, SW59 SW_MEC_5G, SW6 SW_MEC_5G, SW60 SW_MEC_5G, SW61 SW_MEC_5G, SW62 SW_MEC_5G, SW63 SW_MEC_5G, SW64 SW_MEC_5G, SW65 SW_MEC_5G, SW66 SW_MEC_5G, SW67 SW_MEC_5G, SW68 SW_MEC_5G, SW69 SW_MEC_5G, SW7 SW_MEC_5G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

Commit message: Chenged the chematic switches to mx-switches
Parts:
- removed SW1, SW10, SW104, SW105, SW106, SW108, SW11, SW12, SW13, SW14, SW15, SW16, SW17, SW18, SW19, SW2, SW21, SW22, SW23, SW24, SW25, SW26, SW27, SW28, SW29, SW3, SW31, SW32, SW33, SW34, SW35, SW36, SW37, SW38, SW39, SW4, SW41, SW42, SW43, SW44, SW45, SW46, SW47, SW48, SW49, SW5, SW55, SW56, SW57, SW58, SW59, SW6, SW60, SW61, SW62, SW63, SW64, SW65, SW66, SW67, SW68, SW7, SW70, SW71, SW72, SW73, SW74, SW75, SW76, SW77, SW78, SW79, SW8, SW81, SW82, SW83, SW84, SW85, SW86, SW88, SW89, SW9, SW91, SW92, SW93, SW94, SW96, SW97, SW98, SW99: SW_MEC_5G, Button_Switch_Keyboard:SW_Cherry_MX_1.00u_PCB, symbol Switch:SW_MEC_5G
- removed SW100, SW87: SW_MEC_5G, Button_Switch_Keyboard:SW_Cherry_MX_2.00u_Vertical_PCB, symbol Switch:SW_MEC_5G
- removed SW101, SW102, SW103, SW50, SW51, SW52, SW54: SW_MEC_5G, Button_Switch_Keyboard:SW_Cherry_MX_1.25u_PCB, symbol Switch:SW_MEC_5G
- removed SW107, SW69: SW_MEC_5G, Button_Switch_Keyboard:SW_Cherry_MX_2.00u_PCB, symbol Switch:SW_MEC_5G
- removed SW20, SW80: SW_MEC_5G, Button_Switch_Keyboard:SW_Cherry_MX_1.50u_PCB, symbol Switch:SW_MEC_5G
- removed SW30: SW_MEC_5G, Button_Switch_Keyboard:SW_Cherry_MX_1.75u_PCB, symbol Switch:SW_MEC_5G
- removed SW40, SW90: SW_MEC_5G, Button_Switch_Keyboard:SW_Cherry_MX_2.25u_PCB, symbol Switch:SW_MEC_5G
- removed SW53: SW_MEC_5G, Button_Switch_Keyboard:SW_Cherry_MX_6.25u_PCB, symbol Switch:SW_MEC_5G
- removed SW95: SW_MEC_5G, Button_Switch_Keyboard:SW_Cherry_MX_2.75u_PCB, symbol Switch:SW_MEC_5G
- added MX1, MX10, MX100, MX104, MX105, MX106, MX107, MX108, MX11, MX12, MX13, MX14, MX15, MX16, MX17, MX18, MX19, MX2, MX21, MX22, MX23, MX24, MX25, MX26, MX27, MX28, MX29, MX3, MX31, MX32, MX33, MX34, MX35, MX36, MX37, MX38, MX39, MX4, MX40, MX41, MX42, MX43, MX44, MX45, MX46, MX47, MX48, MX49, MX5, MX53, MX55, MX56, MX57, MX58, MX59, MX6, MX60, MX61, MX62, MX63, MX64, MX65, MX66, MX67, MX68, MX69, MX7, MX70, MX71, MX72, MX73, MX74, MX75, MX76, MX77, MX78, MX79, MX8, MX81, MX82, MX83, MX84, MX85, MX86, MX87, MX88, MX89, MX9, MX90, MX91, MX92, MX93, MX94, MX95, MX96, MX97, MX98, MX99: MX_SW_solder, PCM_marbastlib-mx:SW_MX_1u, symbol PCM_marbastlib-mx:MX_SW_solder
- added MX101, MX102, MX50, MX51, MX52, MX54: MX_SW_solder, PCM_marbastlib-mx:SW_MX_1.25u, symbol PCM_marbastlib-mx:MX_SW_solder
- added MX103: MX_SW_solder, PCM_marbastlib-mx:SW_MX_HS_1.25u, symbol PCM_marbastlib-mx:MX_SW_solder
- added MX20: MX_SW_solder, PCM_marbastlib-mx:SW_MX_HS_1.5u, symbol PCM_marbastlib-mx:MX_SW_solder
- added MX30: MX_SW_solder, PCM_marbastlib-mx:SW_MX_1.75u, symbol PCM_marbastlib-mx:MX_SW_solder
- added MX80: MX_SW_solder, PCM_marbastlib-mx:SW_MX_1.5u, symbol PCM_marbastlib-mx:MX_SW_solder
Connections:
- net OUT0: now also MX1.2, MX2.2, MX3.2, MX4.2, MX5.2, MX6.2, MX7.2, MX8.2, MX9.2
- net OUT1: now also MX10.2, MX11.2, MX12.2, MX13.2, MX14.2, MX15.2, MX16.2, MX17.2, MX18.2, MX19.2
- net OUT10: now also MX100.2, MX94.2, MX95.2, MX96.2, MX97.2, MX98.2, MX99.2
- net OUT11: now also MX101.2, MX102.2, MX103.2, MX104.2, MX105.2, MX106.2, MX107.2, MX108.2
- net OUT2: now also MX20.2, MX21.2, MX22.2, MX23.2, MX24.2, MX25.2, MX26.2, MX27.2, MX28.2, MX29.2
- net OUT3: now also MX30.2, MX31.2, MX32.2, MX33.2, MX34.2, MX35.2, MX36.2, MX37.2, MX38.2, MX39.2
- net OUT4: now also MX40.2, MX41.2, MX42.2, MX43.2, MX44.2, MX45.2, MX46.2, MX47.2, MX48.2, MX49.2
- net OUT5: now also MX50.2, MX51.2, MX52.2, MX53.2, MX54.2
- net OUT6: now also MX55.2, MX56.2, MX57.2, MX58.2, MX59.2, MX60.2, MX61.2, MX62.2, MX63.2, MX64.2, MX65.2
- net OUT7: now also MX66.2, MX67.2, MX68.2, MX69.2, MX70.2, MX71.2, MX72.2, MX73.2, MX74.2, MX75.2, MX76.2
- net OUT8: now also MX77.2, MX78.2, MX79.2, MX80.2, MX81.2, MX82.2, MX83.2, MX84.2, MX85.2, MX86.2, MX87.2
- net OUT9: now also MX88.2, MX89.2, MX90.2, MX91.2, MX92.2, MX93.2
- net at D92.1 (K): now also MX92.1
- net at D42.1 (K): now also MX42.1
- net at D2.1 (K): now also MX2.1
- net at D20.1 (K): now also MX20.1
- net at D97.1 (K): now also MX97.1
- net at D99.1 (K): now also MX99.1
- net at D107.1 (K): now also MX107.1
- net at D21.1 (K): now also MX21.1
- net at D61.1 (K): now also MX61.1
- net at D105.1 (K): now also MX105.1
- net at D7.1 (K): now also MX7.1
- net at D54.1 (K): now also MX54.1
- net at D38.1 (K): now also MX38.1
- net at D93.1 (K): now also MX93.1
- net at D76.1 (K): now also MX76.1
- net at D44.1 (K): now also MX44.1
- net at D95.1 (K): now also MX95.1
- net at D39.1 (K): now also MX39.1
- net at D90.1 (K): now also MX90.1
- net at D81.1 (K): now also MX81.1
- net at D46.1 (K): now also MX46.1
- net at D86.1 (K): now also MX86.1
- net at D94.1 (K): now also MX94.1
- net at D9.1 (K): now also MX9.1
- net at D68.1 (K): now also MX68.1
- net at D80.1 (K): now also MX80.1
- net at D84.1 (K): now also MX84.1
- net at D35.1 (K): now also MX35.1
- net at D16.1 (K): now also MX16.1
- net at D60.1 (K): now also MX60.1
- net at D12.1 (K): now also MX12.1
- net at D45.1 (K): now also MX45.1
- net at D85.1 (K): now also MX85.1
- net at D63.1 (K): now also MX63.1
- net at D75.1 (K): now also MX75.1
- net at D98.1 (K): now also MX98.1
- net at D15.1 (K): now also MX15.1
- net at D41.1 (K): now also MX41.1
- net at D52.1 (K): now also MX52.1
- net at D96.1 (K): now also MX96.1
- net at D33.1 (K): now also MX33.1
- net at D19.1 (K): now also MX19.1
- net at D58.1 (K): now also MX58.1
- net at D65.1 (K): now also MX65.1
- net at D53.1 (K): now also MX53.1
- net at D74.1 (K): now also MX74.1
- net at D3.1 (K): now also MX3.1
- net at D108.1 (K): now also MX108.1
- net at D34.1 (K): now also MX34.1
- net at D37.1 (K): now also MX37.1
- net at D67.1 (K): now also MX67.1
- net at D47.1 (K): now also MX47.1
- net at D88.1 (K): now also MX88.1
- net at D49.1 (K): now also MX49.1
- net at D73.1 (K): now also MX73.1
- net at D78.1 (K): now also MX78.1
- net at D24.1 (K): now also MX24.1
- net at D56.1 (K): now also MX56.1
- net at D11.1 (K): now also MX11.1
- net at D43.1 (K): now also MX43.1
- net at D106.1 (K): now also MX106.1
- net at D70.1 (K): now also MX70.1
- net at D29.1 (K): now also MX29.1
- net at D57.1 (K): now also MX57.1
- net at D22.1 (K): now also MX22.1
- net at D72.1 (K): now also MX72.1
- net at D32.1 (K): now also MX32.1
- net at D89.1 (K): now also MX89.1
- net at D4.1 (K): now also MX4.1
- net at D104.1 (K): now also MX104.1
- net at D31.1 (K): now also MX31.1
- net at D25.1 (K): now also MX25.1
- net at D6.1 (K): now also MX6.1
- net at D36.1 (K): now also MX36.1
- net at D62.1 (K): now also MX62.1
- net at D66.1 (K): now also MX66.1
- net at D103.1 (K): now also MX103.1
- net at D102.1 (K): now also MX102.1
- net at D40.1 (K): now also MX40.1
- net at D28.1 (K): now also MX28.1
- net at D50.1 (K): now also MX50.1
- net at D26.1 (K): now also MX26.1
- net at D30.1 (K): now also MX30.1
- net at D55.1 (K): now also MX55.1
- net at D8.1 (K): now also MX8.1
- net at D77.1 (K): now also MX77.1
- net at D101.1 (K): now also MX101.1
- net at D14.1 (K): now also MX14.1
- net at D82.1 (K): now also MX82.1
- net at D87.1 (K): now also MX87.1
- net at D69.1 (K): now also MX69.1
- net at D51.1 (K): now also MX51.1
- net at D1.1 (K): now also MX1.1
- net at D71.1 (K): now also MX71.1
- net at D18.1 (K): now also MX18.1
- net at D13.1 (K): now also MX13.1
- net at D10.1 (K): now also MX10.1
- net at D59.1 (K): now also MX59.1
- net at D17.1 (K): now also MX17.1
- net at D79.1 (K): now also MX79.1
- net at D5.1 (K): now also MX5.1
- net at D83.1 (K): now also MX83.1
- net at D64.1 (K): now also MX64.1
- net at D23.1 (K): now also MX23.1
- net at D48.1 (K): now also MX48.1
- net at D91.1 (K): now also MX91.1
- net at D100.1 (K): now also MX100.1
- net at D27.1 (K): now also MX27.1

Commit message: Placed large portion of the diodes
Parts:
- MX103: footprint PCM_marbastlib-mx:SW_MX_HS_1.25u -> PCM_marbastlib-mx:SW_MX_1.25u
- MX20: footprint PCM_marbastlib-mx:SW_MX_HS_1.5u -> PCM_marbastlib-mx:SW_MX_1.5u
- P1: footprint Connector_USB:USB_C_Receptacle_GCT_USB4135-GF-A_6P_TopMnt_Horizontal -> Connector_USB:USB_C_Receptacle_G-Switch_GT-USB-7010ASV
- S2, S5: footprint PCM_marbastlib-mx:STAB_MX_2u -> PCM_marbastlib-mx:STAB_MX_P_2.25u
- S3, S4, S7, S8: footprint PCM_marbastlib-mx:STAB_MX_2u -> PCM_marbastlib-mx:STAB_MX_P_2u
- S6: footprint PCM_marbastlib-mx:STAB_MX_2u -> PCM_marbastlib-mx:STAB_MX_P_2.75u
Other:
- moved on the sheet: MX101, MX102, MX103, MX104, MX105, MX106, MX107, MX108, MX55, MX56, MX57, MX58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

Commit message: placed the rp2040 inside the board
Changed lines of the file:
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@@
       (effects (font (size 1.27 1.27)) (justify right))
     )
-    (property "Value" "MX_SW_solder" (at 389.89 166.37 90)
+    (property "Value" "MX_SW_solder" (at 377.825 166.37 90)
       (effects (font (size 1.27 1.27)) (justify left))
     )
@@
       (effects (font (size 1.27 1.27)) (justify right))
     )
-    (property "Value" "MX_SW_solder" (at 389.89 147.32 90)
+    (property "Value" "MX_SW_solder" (at 375.92 147.32 90)
       (effects (font (size 1.27 1.27)) (justify left))
     )
@@
       (effects (font (size 1.27 1.27)) (justify right))
     )
-    (property "Value" "MX_SW_solder" (at 389.89 222.25 90)
+    (property "Value" "MX_SW_solder" (at 377.19 222.25 90)
       (effects (font (size 1.27 1.27)) (justify left))
     )
@@
       (effects (font (size 1.27 1.27)) (justify right))
     )
-    (property "Value" "MX_SW_solder" (at 389.89 185.42 90)
+    (property "Value" "MX_SW_solder" (at 377.19 185.42 90)
       (effects (font (size 1.27 1.27)) (justify left))
     )

Commit message: Placed and connected all components
Parts:
- removed C3: 100n, Capacitor_SMD:C_0603_1608Metric, symbol Device:C
Connections:
- net SWDCLK is gone; now on net SWCLK: J1.2 (Pin_2)
Changed lines of the file:
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@@
   (junction (at 304.8 106.045) (diameter 0) (color 0 0 0 0)
   )
-  (junction (at 99.06 36.83) (diameter 0) (color 0 0 0 0)
-  )
   (junction (at 121.92 29.21) (diameter 0) (color 0 0 0 0)
   )
@@
   (junction (at 221.615 161.29) (diameter 0) (color 0 0 0 0)
   )
-  (junction (at 91.44 29.21) (diameter 0) (color 0 0 0 0)
-  )
   (junction (at 77.47 34.29) (diameter 0) (color 0 0 0 0)
   )
@@
     (stroke (width 0) (type default))
   )
-  (wire (pts (xy 77.47 29.21) (xy 91.44 29.21))
-    (stroke (width 0) (type default))
-  )
   (wire (pts (xy 74.93 40.64) (xy 74.93 45.72))
     (stroke (width 0) (type default))
@@
     (stroke (width 0) (type default))
   )
-  (wire (pts (xy 91.44 36.83) (xy 99.06 36.83))
-    (stroke (width 0) (type default))
-  )
   (wire (pts (xy 321.31 86.995) (xy 337.82 86.995))
     (stroke (width 0) (type default))
@@
     (stroke (width 0) (type default))
   )
-  (wire (pts (xy 91.44 29.21) (xy 99.06 29.21))
+  (wire (pts (xy 77.47 29.21) (xy 99.06 29.21))
     (stroke (width 0) (type default))
   )
@@
     (effects (font (size 1.27 1.27)) (justify right bottom))
   )
-  (label "SWDCLK" (at 130.81 118.11 0) (fields_autoplaced)
+  (label "SWCLK" (at 130.81 118.11 0) (fields_autoplaced)
     (effects (font (size 1.27 1.27)) (justify left bottom))
   )
@@
         )
       )
-    )
-  )
-  (symbol (lib_id "Device:C") (at 91.44 33.02 0) (unit 1)
-    (in_bom yes) (on_board yes) (dnp no)
-    (property "Reference" "C3" (at 92.71 30.48 0)
-      (effects (font (size 1.27 1.27)) (justify left))
-    )
-    (property "Value" "100n" (at 92.71 35.56 0)
-      (effects (font (size 1.27 1.27)) (justify left))
-    )
-    (property "Footprint" "Capacitor_SMD:C_0603_1608Metric" (at 92.4052 36.83 0)
-      (effects (font (size 1.27 1.27)) hide)
-    )
-    (property "Datasheet" "~" (at 91.44 33.02 0)
-      (effects (font (size 1.27 1.27)) hide)
-    )
-    (pin "1")
-    (pin "2")
-    (instances
-      (project "main_board_schematic"
-        (path "/eeca1343-c7ac-4fd3-9bdf-4d43c95df1aa"
-          (reference "C3") (unit 1)
-        )
-      )
